File: rn_controller/rn_controller.kicad_sch (KiCad schematic)
At the start: 0 parts

Commit message: Working on part selection.
Other:
- added sheet PCIE_CONN (PCIE_CONN.kicad_sch)
- added sheet PSU (PSU.kicad_sch)
- sheet USB_IC ports: added +3.3V, +5V, 1.05V, PCIE_CLK_N, PCIE_CLK_P, PCIE_CLK_nREQ, PCIE_RX_N, PCIE_RX_P, PCIE_TX_N, PCIE_TX_P, PCIE_nRST; removed none
Changed lines of the file:
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@@
 (kicad_sch (version 20230121) (generator eeschema)
   (paper "A4")
-  (sheet (at 204.47 59.69) (size 39.37 20.32) (fields_autoplaced)
+  (wire (pts (xy 116.84 77.47) (xy 110.49 77.47))
+    (stroke (width 0) (type default))
+  )
+  (wire (pts (xy 116.84 109.22) (xy 139.7 109.22))
+    (stroke (width 0) (type default))
+  )
+  (wire (pts (xy 116.84 106.68) (xy 139.7 106.68))
+    (stroke (width 0) (type default))
+  )
+  (wire (pts (xy 139.7 73.66) (xy 163.83 73.66))
+    (stroke (width 0) (type default))
+  )
+  (wire (pts (xy 106.68 73.66) (xy 116.84 73.66))
+    (stroke (width 0) (type default))
+  )
+  (wire (pts (xy 106.68 92.71) (xy 106.68 73.66))
+    (stroke (width 0) (type default))
+  )
+  (wire (pts (xy 139.7 77.47) (xy 160.02 77.47))
+    (stroke (width 0) (type default))
+  )
+  (wire (pts (xy 163.83 73.66) (xy 163.83 92.71))
+    (stroke (width 0) (type default))
+  )
+  (wire (pts (xy 110.49 77.47) (xy 110.49 92.71))
+    (stroke (width 0) (type default))
+  )
+  (wire (pts (xy 160.02 77.47) (xy 160.02 92.71))
+    (stroke (width 0) (type default))
+  )
+  (wire (pts (xy 139.7 68.58) (xy 167.64 68.58))
+    (stroke (width 0) (type default))
+  )
+  (wire (pts (xy 116.84 100.33) (xy 139.7 100.33))
+    (stroke (width 0) (type default))
+  )
+  (wire (pts (xy 116.84 102.87) (xy 139.7 102.87))
+    (stroke (width 0) (type default))
+  )
+  (wire (pts (xy 167.64 68.58) (xy 167.64 92.71))
+    (stroke (width 0) (type default))
+  )
+  (sheet (at 95.25 92.71) (size 21.59 34.29) (fields_autoplaced)
     (stroke (width 0.1524) (type solid))
     (fill (color 0 0 0 0.0000))
-    (property "Sheetname" "USB_IC" (at 204.47 58.9784 0)
+    (property "Sheetname" "PCIE_CONN" (at 95.25 91.9984 0)
       (effects (font (size 1.27 1.27)) (justify left bottom))
     )
-    (property "Sheetfile" "USB_IC.kicad_sch" (at 204.47 80.5946 0)
+    (property "Sheetfile" "PCIE_CONN.kicad_sch" (at 95.25 127.5846 0)
       (effects (font (size 1.27 1.27)) (justify left top))
+    )
+    (pin "PCIE_N_RESET" output (at 116.84 121.92 0)
+      (effects (font (size 1.27 1.27)) (justify right))
+    )
+    (pin "PCIE_CLK_REQ" output (at 116.84 124.46 0)
+      (effects (font (size 1.27 1.27)) (justify right))
+    )
+    (pin "PCIE_RX_P" output (at 116.84 106.68 0)
+      (effects (font (size 1.27 1.27)) (justify right))
+    )
+    (pin "PCIE_RX_N" output (at 116.84 109.22 0)
+      (effects (font (size 1.27 1.27)) (justify right))
+    )
+    (pin "PCIE_TX_P" output (at 116.84 113.03 0)
+      (effects (font (size 1.27 1.27)) (justify right))
+    )
+    (pin "PCIE_TX_N" output (at 116.84 115.57 0)
+      (effects (font (size 1.27 1.27)) (justify right))
+    )
+    (pin "PCIE_CLK_P" output (at 116.84 100.33 0)
+      (effects (font (size 1.27 1.27)) (justify right))
+    )
+    (pin "PCIE_CLK_N" output (at 116.84 102.87 0)
+      (effects (font (size 1.27 1.27)) (justify right))
+    )
+    (pin "3.3v" output (at 106.68 92.71 90)
+      (effects (font (size 1.27 1.27)) (justify right))
+    )
+    (pin "12v" output (at 110.49 92.71 90)
+      (effects (font (size 1.27 1.27)) (justify right))
+    )
+    (instances
+      (project "rn_controller"
+        (path "/4627b6c4-e89d-474f-b44e-65b603588291" (page "3"))
+      )
+    )
+  )
+  (sheet (at 139.7 92.71) (size 39.37 34.29) (fields_autoplaced)
+    (stroke (width 0.1524) (type solid))
+    (fill (color 0 0 0 0.0000))
+    (property "Sheetname" "USB_IC" (at 139.7 91.9984 0)
+      (effects (font (size 1.27 1.27)) (justify left bottom))
+    )
+    (property "Sheetfile" "USB_IC.kicad_sch" (at 139.7 127.5846 0)
+      (effects (font (size 1.27 1.27)) (justify left top))
+    )
+    (pin "PCIE_CLK_N" input (at 139.7 102.87 180)
+      (effects (font (size 1.27 1.27)) (justify left))
+    )
+    (pin "PCIE_TX_N" input (at 139.7 115.57 180)
+      (effects (font (size 1.27 1.27)) (justify left))
+    )
+    (pin "PCIE_nRST" input (at 139.7 121.92 180)
+      (effects (font (size 1.27 1.27)) (justify left))
+    )
+    (pin "PCIE_CLK_nREQ" input (at 139.7 124.46 180)
+      (effects (font (size 1.27 1.27)) (justify left))
+    )
+    (pin "PCIE_TX_P" input (at 139.7 113.03 180)
+      (effects (font (size 1.27 1.27)) (justify left))
+    )
+    (pin "PCIE_CLK_P" input (at 139.7 100.33 180)
+      (effects (font (size 1.27 1.27)) (justify left))
+    )
+    (pin "PCIE_RX_P" input (at 139.7 106.68 180)
+      (effects (font (size 1.27 1.27)) (justify left))
+    )
+    (pin "PCIE_RX_N" input (at 139.7 109.22 180)
+      (effects (font (size 1.27 1.27)) (justify left))
+    )
+    (pin "+3.3V" input (at 160.02 92.71 90)
+      (effects (font (size 1.27 1.27)) (justify right))
+    )
+    (pin "1.05V" input (at 163.83 92.71 90)
+      (effects (font (size 1.27 1.27)) (justify right))
+    )
+    (pin "+5V" input (at 167.64 92.71 90)
+      (effects (font (size 1.27 1.27)) (justify right))
     )
     (instances
@@
       )
     )
+  )
+  (sheet (at 116.84 66.04) (size 22.86 16.51) (fields_autoplaced)
+    (stroke (width 0.1524) (type solid))
+    (fill (color 0 0 0 0.0000))
+    (property "Sheetname" "PSU" (at 116.84 65.3284 0)
+      (effects (font (size 1.27 1.27)) (justify left bottom))
+    )
+    (property "Sheetfile" "PSU.kicad_sch" (at 116.84 83.1346 0)
+      (effects (font (size 1.27 1.27)) (justify left top))
+    )
+    (pin "12V" output (at 116.84 77.47 180)
+      (effects (font (size 1.27 1.27)) (justify left))
+    )
+    (pin "3.3V" output (at 116.84 73.66 180)
+      (effects (font (size 1.27 1.27)) (justify left))
+    )
+    (pin "1.05V" output (at 139.7 73.66 0)
+      (effects (font (size 1.27 1.27)) (justify right))
+    )
+    (pin "5V" output (at 139.7 68.58 0)
+      (effects (font (size 1.27 1.27)) (justify right))
+    )
+    (pin "3.3Vout" output (at 139.7 77.47 0)
+      (effects (font (size 1.27 1.27)) (justify right))
+    )
+    (instances
+      (project "rn_controller"
+        (path "/4627b6c4-e89d-474f-b44e-65b603588291" (page "4"))
+      )
+    )

Commit message: Finished routing.
Changed lines of the file:
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@@
 (kicad_sch (version 20230121) (generator eeschema)
   (paper "A4")
+  (wire (pts (xy 116.84 124.46) (xy 139.7 124.46))
+    (stroke (width 0) (type default))
+  )
   (wire (pts (xy 116.84 77.47) (xy 110.49 77.47))
     (stroke (width 0) (type default))
@@
     (stroke (width 0) (type default))
   )
+  (wire (pts (xy 116.84 121.92) (xy 139.7 121.92))
+    (stroke (width 0) (type default))
+  )
+  (wire (pts (xy 116.84 115.57) (xy 139.7 115.57))
+    (stroke (width 0) (type default))
+  )
   (wire (pts (xy 160.02 77.47) (xy 160.02 92.71))
     (stroke (width 0) (type default))
@@
     (stroke (width 0) (type default))
   )
+  (wire (pts (xy 116.84 113.03) (xy 139.7 113.03))
+    (stroke (width 0) (type default))
+  )
