File: rn_controller/PSU.kicad_sch (KiCad schematic)
At the start: 13 parts, among them U2 LM2596S-5, U3 TLV743105PDBVR

Commit message: Finished routing.
Parts:
- removed D1: 1N5824, symbol Device:D_Zener
- removed L1: 33uH, symbol Device:L
- added D1: SS34-MS, NEW:DO-214AC_L4.3-W2.7-LS5.0-RD, symbol NEW:SS34-MS
- added L2: FXL0650-330-M, NEW:IND-SMD_L7.0-W6.6_FXL0650, symbol NEW:FXL0650-330-M
- C22: footprint (none) -> Capacitor_SMD:CP_Elec_6.3x7.7; LCSC Part (none) -> C497598
- C23: footprint (none) -> Capacitor_SMD:CP_Elec_10x10.5; LCSC Part (none) -> C497598
- C24, C25: footprint (none) -> Resistor_SMD:R_0402_1005Metric; LCSC Part (none) -> C77006
Connections:
- net GND: now also D1.2 (K)
- net at C22.1, R10.1, U2.4 (FB): now also L2.2
- net at U2.2 (OUT): now also D1.1 (A), L2.1
Changed lines of the file:
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@@
 (kicad_sch (version 20230121) (generator eeschema)
   (paper "A4")
-  (junction (at 161.29 77.47) (diameter 0) (color 0 0 0 0)
+  (junction (at 160.02 77.47) (diameter 0) (color 0 0 0 0)
   )
   (junction (at 127 121.92) (diameter 0) (color 0 0 0 0)
@@
     (stroke (width 0) (type default))
   )
-  (wire (pts (xy 161.29 77.47) (xy 153.67 77.47))
-    (stroke (width 0) (type default))
-  )
-  (wire (pts (xy 166.37 77.47) (xy 161.29 77.47))
+  (wire (pts (xy 153.67 77.47) (xy 160.02 77.47))
     (stroke (width 0) (type default))
   )
@@
     (stroke (width 0) (type default))
   )
+  (wire (pts (xy 160.02 77.47) (xy 166.37 77.47))
+    (stroke (width 0) (type default))
+  )
   (wire (pts (xy 179.07 113.03) (xy 190.5 113.03))
     (stroke (width 0) (type default))
@@
     (stroke (width 0) (type default))
   )
-  (wire (pts (xy 181.61 77.47) (xy 173.99 77.47))
+  (wire (pts (xy 181.61 77.47) (xy 176.53 77.47))
     (stroke (width 0) (type default))
   )
@@
       (effects (font (size 1.27 1.27)) (justify left))
     )
-    (property "Footprint" "" (at 110.1852 80.01 0)
+    (property "Footprint" "Capacitor_SMD:CP_Elec_10x10.5" (at 110.1852 80.01 0)
       (effects (font (size 1.27 1.27)) hide)
     )
@@
       (effects (font (size 1.27 1.27)) hide)
     )
+    (property "LCSC Part" "C497598" (at 109.22 76.2 0)
+      (effects (font (size 1.27 1.27)) hide)
+    )
     (pin "1")
     (pin "2")
@@
     )
   )
+  (symbol (lib_id "NEW:SS34-MS") (at 160.02 82.55 270) (unit 1)
+    (in_bom yes) (on_board yes) (dnp no) (fields_autoplaced)
+    (property "Reference" "D1" (at 162.56 81.28 90)
+      (effects (font (size 1.27 1.27)) (justify left))
+    )
+    (property "Value" "SS34-MS" (at 162.56 83.82 90)
+      (effects (font (size 1.27 1.27)) (justify left))
+    )
+    (property "Footprint" "NEW:DO-214AC_L4.3-W2.7-LS5.0-RD" (at 152.4 82.55 0)
+      (effects (font (size 1.27 1.27)) hide)
+    )
+    (property "Datasheet" "" (at 160.02 82.55 0)
+      (effects (font (size 1.27 1.27)) hide)
+    )
+    (property "LCSC Part" "C2836396" (at 149.86 82.55 0)
+      (effects (font (size 1.27 1.27)) hide)
+    )
+    (pin "1")
+    (pin "2")
+    (instances
+      (project "rn_controller"
+        (path "/4627b6c4-e89d-474f-b44e-65b603588291/c856299a-2981-4be4-929c-355b69c9e9df"
+          (reference "D1") (unit 1)
+        )
+      )
+    )
+  )
   (symbol (lib_id "Device:C_Polarized") (at 181.61 81.28 0) (unit 1)
     (in_bom yes) (on_board yes) (dnp no) (fields_autoplaced)
@@
       (effects (font (size 1.27 1.27)) (justify left))
     )
-    (property "Footprint" "" (at 182.5752 85.09 0)
+    (property "Footprint" "Capacitor_SMD:CP_Elec_6.3x7.7" (at 182.5752 85.09 0)
       (effects (font (size 1.27 1.27)) hide)
     )
     (property "Datasheet" "~" (at 181.61 81.28 0)
+      (effects (font (size 1.27 1.27)) hide)
+    )
+    (property "LCSC Part" "C497598" (at 181.61 81.28 0)
       (effects (font (size 1.27 1.27)) hide)
     )
@@
       (effects (font (size 1.27 1.27)) (justify left))
     )
-    (property "Footprint" "" (at 122.8852 134.62 0)
+    (property "Footprint" "Resistor_SMD:R_0402_1005Metric" (at 122.8852 134.62 0)
       (effects (font (size 1.27 1.27)) hide)
     )
@@
       (effects (font (size 1.27 1.27)) hide)
     )
+    (property "LCSC Part" "C77006" (at 121.92 130.81 0)
+      (effects (font (size 1.27 1.27)) hide)
+    )
     (pin "1")
     (pin "2")
@@
         (path "/4627b6c4-e89d-474f-b44e-65b603588291/c856299a-2981-4be4-929c-355b69c9e9df"
           (reference "C24") (unit 1)
-        )
-      )
-    )
-  )
-  (symbol (lib_id "Device:L") (at 170.18 77.47 90) (unit 1)
-    (in_bom yes) (on_board yes) (dnp no)
-    (property "Reference" "L1" (at 170.18 74.93 90)
-      (effects (font (size 1.27 1.27)))
-    )
-    (property "Value" "33uH" (at 170.18 78.74 90)
-      (effects (font (size 1.27 1.27)))
-    )
-    (property "Footprint" "" (at 170.18 77.47 0)
-      (effects (font (size 1.27 1.27)) hide)
-    )
-    (property "Datasheet" "~" (at 170.18 77.47 0)
-      (effects (font (size 1.27 1.27)) hide)
-    )
-    (pin "1")
-    (pin "2")
-    (instances
-      (project "rn_controller"
-        (path "/4627b6c4-e89d-474f-b44e-65b603588291/c856299a-2981-4be4-929c-355b69c9e9df"
-          (reference "L1") (unit 1)
         )
       )
@@
     )
   )
-  (symbol (lib_id "Device:D_Zener") (at 161.29 81.28 270) (unit 1)
-    (in_bom yes) (on_board yes) (dnp no) (fields_autoplaced)
-    (property "Reference" "D1" (at 163.83 80.01 90)
-      (effects (font (size 1.27 1.27)) (justify left))
-    )
-    (property "Value" "1N5824" (at 163.83 82.55 90)
-      (effects (font (size 1.27 1.27)) (justify left))
-    )
-    (property "Footprint" "" (at 161.29 81.28 0)
-      (effects (font (size 1.27 1.27)) hide)
-    )
-    (property "Datasheet" "~" (at 161.29 81.28 0)
-      (effects (font (size 1.27 1.27)) hide)
-    )
-    (pin "1")
-    (pin "2")
-    (instances
-      (project "rn_controller"
-        (path "/4627b6c4-e89d-474f-b44e-65b603588291/c856299a-2981-4be4-929c-355b69c9e9df"
-          (reference "D1") (unit 1)
-        )
-      )
-    )
-  )
   (symbol (lib_id "Device:R") (at 128.27 86.36 0) (unit 1)
     (in_bom yes) (on_board yes) (dnp no) (fields_autoplaced)
@@
     )
   )
-  (symbol (lib_id "power:GND") (at 161.29 85.09 0) (unit 1)
-    (in_bom yes) (on_board yes) (dnp no) (fields_autoplaced)
-    (property "Reference" "#PWR09" (at 161.29 91.44 0)
-      (effects (font (size 1.27 1.27)) hide)
-    )
-    (property "Value" "GND" (at 161.29 90.17 0)
-      (effects (font (size 1.27 1.27)))
-    )
-    (property "Footprint" "" (at 161.29 85.09 0)
-      (effects (font (size 1.27 1.27)) hide)
-    )
-    (property "Datasheet" "" (at 161.29 85.09 0)
+  (symbol (lib_id "power:GND") (at 160.02 87.63 0) (unit 1)
+    (in_bom yes) (on_board yes) (dnp no) (fields_autoplaced)
+    (property "Reference" "#PWR09" (at 160.02 93.98 0)
+      (effects (font (size 1.27 1.27)) hide)
+    )
+    (property "Value" "GND" (at 160.02 92.71 0)
+      (effects (font (size 1.27 1.27)))
+    )
+    (property "Footprint" "" (at 160.02 87.63 0)
+      (effects (font (size 1.27 1.27)) hide)
+    )
+    (property "Datasheet" "" (at 160.02 87.63 0)
       (effects (font (size 1.27 1.27)) hide)
     )
@@
     )
   )
+  (symbol (lib_id "NEW:FXL0650-330-M") (at 171.45 77.47 0) (unit 1)
+    (in_bom yes) (on_board yes) (dnp no) (fields_autoplaced)
+    (property "Reference" "L2" (at 171.45 71.12 0)
+      (effects (font (size 1.27 1.27)))
+    )
+    (property "Value" "FXL0650-330-M" (at 171.45 73.66 0)
+      (effects (font (size 1.27 1.27)))
+    )
+    (property "Footprint" "NEW:IND-SMD_L7.0-W6.6_FXL0650" (at 171.45 85.09 0)
+      (effects (font (size 1.27 1.27)) hide)
+    )
+    (property "Datasheet" "https://lcsc.com/product-detail/Power-Inductors_cjiang-Changjiang-Microelectronics-Tech-FXL0650-330-M_C475526.html" (at 171.45 87.63 0)
+      (effects (font (size 1.27 1.27)) hide)
+    )
+    (property "LCSC Part" "C475526" (at 171.45 90.17 0)
+      (effects (font (size 1.27 1.27)) hide)
+    )
+    (pin "1")
+    (pin "2")
+    (instances
+      (project "rn_controller"
+        (path "/4627b6c4-e89d-474f-b44e-65b603588291/c856299a-2981-4be4-929c-355b69c9e9df"
+          (reference "L2") (unit 1)
+        )
+      )
+    )
+  )
   (symbol (lib_id "Device:C") (at 162.56 130.81 0) (unit 1)
     (in_bom yes) (on_board yes) (dnp no) (fields_autoplaced)
@@
       (effects (font (size 1.27 1.27)) (justify left))
     )
-    (property "Footprint" "" (at 163.5252 134.62 0)
+    (property "Footprint" "Resistor_SMD:R_0402_1005Metric" (at 163.5252 134.62 0)
       (effects (font (size 1.27 1.27)) hide)
     )
@@
       (effects (font (size 1.27 1.27)) hide)
     )
+    (property "LCSC Part" "C77006" (at 162.56 130.81 0)
+      (effects (font (size 1.27 1.27)) hide)
+    )

Commit message: Fixed capacitor.
Parts:
- C22: LCSC Part C497598 -> C336314
Changed lines of the file:
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@@
       (effects (font (size 1.27 1.27)) hide)
     )
-    (property "LCSC Part" "C497598" (at 181.61 81.28 0)
+    (property "LCSC Part" "C336314" (at 181.61 81.28 0)
       (effects (font (size 1.27 1.27)) hide)
     )
